File: project/hw/mb/mb.sch (KiCad schematic (older format))
At the start: 18 parts, among them P1 CONN_02X04, P2 CONN_01X05, P3 CONN_01X05, SW1 SW_PUSH, SW2 SW_PUSH, U1 LPC1114/302

Commit message: motherboard design done
Parts:
- removed C10, C3, C5, C7, C8, C9: CP, Capacitors_SMD:c_elec_4x5.7, symbol CP
- removed P3: CONN_01X05, Pin_Headers:Pin_Header_Straight_1x05, symbol CONN_01X05
- added C10, C13, C9: 100n, Capacitors_SMD:C_0805_HandSoldering, symbol C
- added C11, C12, C3, C5, C7, C8: 1u, Capacitors_SMD:C_1206_HandSoldering, symbol C
- added P10, P11, P6, P7, P8, P9: CONN_01X08, Connectors_Molex:Connector_Molex_PicoBlade_53398-0871, symbol CONN_01X08
- added P4, P5: CONN_01X02, Pin_Headers:Pin_Header_Straight_1x02, symbol CONN_01X02
- added R3, R4: 4k7, Resistors_SMD:R_0805_HandSoldering, symbol R
- added R5: 0, Resistors_SMD:R_1206_HandSoldering, symbol R
- added U2: mcp1700, Housings_SOT-23_SOT-143_TSOT-6:SOT-23_Handsoldering, symbol mcp1700
- C4, C6: value C -> 1u; footprint Capacitors_SMD:C_0805_HandSoldering -> Capacitors_SMD:C_1206_HandSoldering
Connections:
- net labels added: IMUA0, IMUA1, IMUA2, IMUA3, IMUA4, IMUA5
- net labels removed: +3.3V
- wire segments 83 -> 131
- no-connect marks 4 -> 41
Other:
- moved on the sheet: C4, C6
