File: project/hw/imu/imu.kicad_pcb (KiCad board)
At the start: 2 copper layers, 12 x 15 mm, 5 parts, among them P1 CONN_5, U1 LIS2HH12_I2C, U2 BMG160_i2c

Commit message: arne
Routing:
- net GND: track 28.3 -> 23.1 mm, vias 1 -> 0
- added copper zone on B.Cu, net GND
Other:
- net class Default: clearance 0.25 -> 0.248; trace_width 0.25 -> 0.248
- rule trace_clearance: 0.25 -> 0.248
- board text added: "IMU board"
Changed lines of the file:
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@@
     (area 109.949999 99.449999 122.050001 114.550001)
     (thickness 1.6)
-    (drawings 9)
-    (tracks 109)
+    (drawings 10)
+    (tracks 104)
     (zones 0)
     (modules 5)
@@
   )
   (setup
-    (last_trace_width 0.25)
-    (trace_clearance 0.25)
+    (last_trace_width 0.248)
+    (user_trace_width 0.8)
+    (trace_clearance 0.248)
     (zone_clearance 0.508)
     (zone_45_only yes)
@@
     (visible_elements FFFFFF7F)
     (pcbplotparams
-      (layerselection 0x00030_80000001)
+      (layerselection 0x01000_80000001)
       (usegerberextensions false)
       (excludeedgelayer true)
@@
       (outputformat 1)
       (mirror false)
-      (drillshape 1)
+      (drillshape 0)
       (scaleselection 1)
-      (outputdirectory ""))
+      (outputdirectory /tmp/gerbers/))
   )
   (net 0 "")
@@
   (net 7 "Net-(U2-Pad5)")
   (net_class Default "This is the default net class."
-    (clearance 0.25)
-    (trace_width 0.25)
+    (clearance 0.248)
+    (trace_width 0.248)
     (via_dia 1.44)
     (via_drill 0.5588)
@@
       (rotate (xyz 0 0 0))
     )
+  )
+  (gr_text "IMU board" (at 116.05 113.16) (layer B.Cu)
+    (effects (font (size 1.5 1.5) (thickness 0.3)) (justify mirror))
   )
   (gr_text 5 (at 120.76 100.49) (layer F.Cu)
@@
   (segment (start 116.42 106.56) (end 116.42 107.06) (width 0.25) (layer F.Cu) (net 1))
   (segment (start 113.12 106.56) (end 116.42 106.56) (width 0.25) (layer F.Cu) (net 1))
-  (segment (start 118 104.56) (end 119.82 104.56) (width 0.25) (layer B.Cu) (net 2))
-  (via (at 120.11 104.85) (size 1.44) (drill 0.5588) (layers F.Cu B.Cu) (net 2))
-  (segment (start 119.82 104.56) (end 120.11 104.85) (width 0.25) (layer B.Cu) (net 2))
+  (segment (start 117.11 104.7) (end 117.27 104.7) (width 0.248) (layer B.Cu) (net 2))
+  (segment (start 116.05 100.904999) (end 114.445001 100.904999) (width 0.25) (layer F.Cu) (net 2))
+  (segment (start 117.280001 101.280001) (end 118 102) (width 0.25) (layer F.Cu) (net 2))
+  (segment (start 116.05 100.904999) (end 116.904999 100.904999) (width 0.25) (layer F.Cu) (net 2))
+  (segment (start 116.904999 100.904999) (end 117.280001 101.280001) (width 0.25) (layer F.Cu) (net 2))
+  (segment (start 114.445001 100.904999) (end 114.19 101.16) (width 0.25) (layer F.Cu) (net 2))
+  (segment (start 114.19 101.16) (end 114.19 103.08) (width 0.25) (layer F.Cu) (net 2))
+  (segment (start 114.19 103.08) (end 114.52 103.41) (width 0.25) (layer F.Cu) (net 2))
   (segment (start 115.77 104.96) (end 115.77 103.75) (width 0.25) (layer F.Cu) (net 2))
+  (segment (start 115.43 103.41) (end 114.52 103.41) (width 0.25) (layer F.Cu) (net 2))
   (segment (start 115.77 103.75) (end 115.43 103.41) (width 0.25) (layer F.Cu) (net 2))
-  (segment (start 115.43 103.41) (end 114.52 103.41) (width 0.25) (layer F.Cu) (net 2))
   (segment (start 116.42 105.56) (end 116.36 105.5) (width 0.25) (layer F.Cu) (net 2))
   (segment (start 116.36 105.5) (end 115.86 105.5) (width 0.25) (layer F.Cu) (net 2))
@@
   (segment (start 115 105.5) (end 115 104.68) (width 0.25) (layer F.Cu) (net 2))
   (segment (start 115 104.68) (end 115.02 104.66) (width 0.25) (layer F.Cu) (net 2))
-  (segment (start 116.904999 100.904999) (end 117.280001 101.280001) (width 0.25) (layer F.Cu) (net 2))
-  (segment (start 114.52 103.41) (end 114.364999 103.254999) (width 0.25) (layer F.Cu) (net 2))
   (segment (start 114.52 104.66) (end 114.52 103.41) (width 0.25) (layer F.Cu) (net 2))
-  (segment (start 114.364999 103.254999) (end 114.364999 101.474399) (width 0.25) (layer F.Cu) (net 2))
-  (segment (start 114.364999 101.474399) (end 114.934399 100.904999) (width 0.25) (layer F.Cu) (net 2))
-  (segment (start 114.934399 100.904999) (end 116.904999 100.904999) (width 0.25) (layer F.Cu) (net 2))
-  (segment (start 117.280001 101.280001) (end 118 102) (width 0.25) (layer F.Cu) (net 2))
   (segment (start 117.11 104.7) (end 117.11 104.825) (width 0.25) (layer B.Cu) (net 2))
-  (segment (start 117.11 104.7) (end 117.86 104.7) (width 0.25) (layer B.Cu) (net 2))
-  (segment (start 117.86 104.7) (end 118 104.56) (width 0.25) (layer B.Cu) (net 2))
-  (segment (start 118 104.56) (end 118 103.91) (width 0.25) (layer B.Cu) (net 2))
   (segment (start 115.78 112.88) (end 115.78 113.255) (width 0.25) (layer F.Cu) (net 2))
-  (segment (start 118 102) (end 118 103.91) (width 0.25) (layer B.Cu) (net 2))
   (segment (start 119.24 113.87) (end 119.63 113.48) (width 0.25) (layer F.Cu) (net 2))
   (segment (start 119.63 113.48) (end 119.63 112.88) (width 0.25) (layer F.Cu) (net 2))
@@
   (segment (start 112.9835 105.4235) (end 113.12 105.56) (width 0.25) (layer F.Cu) (net 4))
   (segment (start 115.78 111.88) (end 114.5 111.88) (width 0.25) (layer F.Cu) (net 4))
-  (segment (start 120.72 101.96) (end 119.905 101.145) (width 0.25) (layer B.Cu) (net 5) (status 400000))
+  (segment (start 120.72 101.96) (end 119.905 101.145) (width 0.25) (layer B.Cu) (net 5))
   (segment (start 116.234999 105.646768) (end 116.234999 104.25) (width 0.25) (layer B.Cu) (net 5))
   (segment (start 116.234999 105.646768) (end 112.9 108.981767) (width 0.25) (layer B.Cu) (net 5))
@@
   (segment (start 119.23 100.47) (end 119.905 101.145) (width 0.25) (layer B.Cu) (net 5))
   (segment (start 116.79 101.99) (end 116.79 101.07) (width 0.25) (layer B.Cu) (net 5))
-  (segment (start 120.72 101.96) (end 120.72 102.06) (width 0.25) (layer B.Cu) (net 5) (status C00000))
+  (segment (start 120.72 101.96) (end 120.72 102.06) (width 0.25) (layer B.Cu) (net 5))
   (segment (start 118.309989 100.404989) (end 119.965 102.06) (width 0.25) (layer F.Cu) (net 5))
-  (segment (start 119.965 102.06) (end 120.72 102.06) (width 0.25) (layer F.Cu) (net 5) (status 800000))
+  (segment (start 119.965 102.06) (end 120.72 102.06) (width 0.25) (layer F.Cu) (net 5))
   (segment (start 114.28 111.38) (end 112.924971 110.024971) (width 0.25) (layer F.Cu) (net 5))
   (segment (start 112.924971 110.024971) (end 112.924971 109.003308) (width 0.25) (layer F.Cu) (net 5))
@@
       )
     )
+  )
+  (zone (net 2) (net_name GND) (layer B.Cu) (hatch edge 0.508)
+    (connect_pads (clearance 0.508))
+    (min_thickness 0.254)
+    (fill yes (arc_segments 16) (thermal_gap 0.508) (thermal_bridge_width 0.508))
+    (polygon
+      (pts
+        (xy 123.79 115.37) (xy 108.97 115.37) (xy 108.97 96.58) (xy 125.0301 96.58) (xy 123.79 115.37)
+      )
+    )
+  )
+  (zone (net 2) (net_name GND) (layer B.Cu) (hatch edge 0.508)
+    (connect_pads (clearance 0.508))
+    (min_thickness 0.254)
+    (fill yes (arc_segments 16) (thermal_gap 0.508) (thermal_bridge_width 0.508))
+    (polygon
+      (pts
+        (xy 125.04 96.43) (xy 125.04 96.58) (xy 125.0301 96.58) (xy 125.04 96.43)
+      )
+    )
